File: RepeatRoverV2.0/RepeatRover.kicad_pcb (KiCad board)
At the start: 2 copper layers, 26 parts, among them J1_1 Conn_01x02_Female, J2_1 Conn_01x02_Female, J3_1 Conn_01x03_Female, J4_1 Conn_01x03_Female, X1 32MHz

Commit message: PCB with revisions from lecture
Parts:
- added C16: 100uF, Capacitor_SMD:C_0805_2012Metric_Pad1.18x1.45mm_HandSolder, F.Cu at (108.0, 74.9)
- added CVIN1: 10uF, Capacitor_SMD:CP_Elec_5x5.7, F.Cu at (90.8, 86.4)
- added CVOUT1: 10uF, Capacitor_SMD:CP_Elec_5x5.7, F.Cu at (90.8, 94.0)
- added C_RST1: 1uF, Capacitor_SMD:C_0805_2012Metric_Pad1.18x1.45mm_HandSolder, F.Cu at (168.9, 123.2)
- added H1: MountingHole, MountingHole:MountingHole_3.2mm_M3, F.Cu at (82.5, 63.5)
- added H2: MountingHole, MountingHole:MountingHole_3.2mm_M3, F.Cu at (177.8, 139.7)
- added H3: MountingHole, MountingHole:MountingHole_3.2mm_M3, F.Cu at (82.5, 139.7)
- added H4: MountingHole, MountingHole:MountingHole_3.2mm_M3, F.Cu at (177.8, 63.5)
- added J5: Barrel_Jack, Connector_BarrelJack:BarrelJack_CUI_PJ-102AH_Horizontal, F.Cu at (93.3, 81.3)
- added LDO1: NCP1117-3.3_SOT223, Package_TO_SOT_SMD:SOT-223-3_TabPin2, F.Cu at (99.7, 88.3)
- added R1: 2.7k, Resistor_SMD:R_0805_2012Metric_Pad1.20x1.40mm_HandSolder, F.Cu at (126.4, 103.5)
- added R2: 2.7k, Resistor_SMD:R_0805_2012Metric_Pad1.20x1.40mm_HandSolder, F.Cu at (129.5, 101.6)
- added R_RST1: 10k, Resistor_SMD:R_0805_2012Metric_Pad1.20x1.40mm_HandSolder, F.Cu at (168.9, 135.9)
- added SW_RST1: _, Button_Switch_THT:SW_PUSH_6mm, F.Cu at (167.0, 132.7)
- X1: footprint Crystal:Crystal_SMD_2016-4Pin_2.0x1.6mm -> Hall Effect Footprint:OSC_XRCGB32M000FXH2CR0
- moved J1_1 71.1 mm to (127.0, 71.8), turned to 0 degrees
- moved C14 65.9 mm to (123.2, 73.0), turned to 90 degrees
- moved J2_1 64.1 mm to (127.0, 78.1), turned to 0 degrees
- moved C13 58.5 mm to (123.2, 79.4), turned to 90 degrees
- moved J3_1 56.5 mm to (149.2, 71.8)
- moved J4_1 56.0 mm to (142.9, 71.8)
- moved U_HB1 55.3 mm to (114.9, 75.6), turned to 0 degrees
- moved C12 50.8 mm to (108.0, 79.4), turned to 270 degrees
- moved L2 46.0 mm to (162.6, 88.3)
- moved L3 44.7 mm to (162.6, 90.8), turned to 270 degrees
- moved C5 44.6 mm to (160.0, 106.0)
- moved C8 44.2 mm to (168.9, 91.4)
- moved MCU1 43.5 mm to (163.8, 99.1)
- moved C2 43.2 mm to (170.8, 91.4)
- moved C4 43.2 mm to (155.6, 96.5)
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Connections:
- C11 pad 2: +3V0 -> +3V3
- MAG1 pad 13: +3V0 -> +3V3
- MAG1 pad 14: Net-(MAG1-Pad12) -> (no net)
- MAG1 pad 15: Net-(MAG1-Pad15) -> (no net)
- MAG1 pad 2: +3V0 -> +3V3
- MAG1 pad 5: (no net) -> Net-(MAG1-Pad5)
- MAG1 pad 6: (no net) -> Net-(MAG1-Pad12)
- MCU1 pad 10: /MISO -> Net-(MCU1-Pad10)
- MCU1 pad 11: Net-(MCU1-Pad11) -> /SCL
- MCU1 pad 12: Net-(MCU1-Pad12) -> /SDA
- MCU1 pad 14: /CS -> Net-(MCU1-Pad14)
- MCU1 pad 21: Net-(MCU1-Pad21) -> /CS
- MCU1 pad 22: /INA -> /MOSI
- MCU1 pad 23: Net-(MCU1-Pad23) -> /SCLK
- MCU1 pad 24: Net-(MCU1-Pad24) -> /MISO
- MCU1 pad 27: /INB -> Net-(MCU1-Pad27)
- MCU1 pad 28: /INC -> Net-(MCU1-Pad28)
- MCU1 pad 29: /IND -> /MSCL
- MCU1 pad 37: /SCL -> Net-(MCU1-Pad37)
- MCU1 pad 38: /SDA -> Net-(MCU1-Pad38)
- MCU1 pad 39: Net-(MCU1-Pad39) -> /WSS1
- MCU1 pad 40: Net-(MCU1-Pad40) -> /WSS2
- MCU1 pad 5: Net-(MCU1-Pad5) -> /INA
- MCU1 pad 6: Net-(MCU1-Pad6) -> /INB
- MCU1 pad 7: Net-(MCU1-Pad7) -> /INC
- MCU1 pad 8: /MOSI -> /IND
- MCU1 pad 9: /SCLK -> Net-(MCU1-Pad9)
- X1 pad 1: /XC2 -> /XC1
- X1 pad 3: /XC1 -> /XC2
Routing:
- net /MISO: track 10.5 -> 90.2 mm, vias 0 -> 2
- net /SCLK: track 12.6 -> 87.4 mm, vias 0 -> 2
- net /MOSI: track 14.9 -> 83.1 mm, vias 0 -> 2
- net /CS: track 25.2 -> 79.7 mm, vias 0 -> 2
- net /INB: track 14.2 -> 63.3 mm, vias 0 -> 2
- net /INC: track 16.2 -> 61.9 mm
- net /MSCL: track 0.00 -> 43.1 mm, vias 0 -> 1
- net /INA: track 21.4 -> 63.9 mm
- net /IND: track 20.3 -> 61.9 mm
- net /WSS1: track 5.09 -> 39.4 mm, vias 1 -> 2
- net (no net): track 32.8 -> 0.00 mm
- net /WSS2: track 13.0 -> 42.4 mm, vias 0 -> 2
- net +6V: track 16.1 -> 45.2 mm, vias 0 -> 3
- net /SCL: track 15.8 -> 41.8 mm
- net GND: track 121.6 -> 99.0 mm, vias 2 -> 0
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
Commit message: new mcu footgprint
Parts:
- removed C3: 0.8pF, Capacitor_SMD:C_0805_2012Metric_Pad1.18x1.45mm_HandSolder
- removed C4, C5, C8: 100nF, Capacitor_SMD:C_0805_2012Metric_Pad1.18x1.45mm_HandSolder
- removed C7: 100pF, Capacitor_SMD:C_0805_2012Metric_Pad1.18x1.45mm_HandSolder
- removed C9: 4.7uF, Capacitor_SMD:C_0805_2012Metric_Pad1.18x1.45mm_HandSolder
- removed L1: 3.9nH, Inductor_SMD:L_0402_1005Metric_Pad0.77x0.64mm_HandSolder
- removed L2: 10uH, Inductor_SMD:L_0201_0603Metric_Pad0.64x0.40mm_HandSolder
- removed L3: 15nH, Inductor_SMD:L_0402_1005Metric_Pad0.77x0.64mm_HandSolder
- removed MCU1: NRF52832-QFAA-R, NRF52832-QFAA-R:QFN40P600X600X90-49N
- added E1: MDBT42Q-512KV2, MDBT42Q-512KV2:RAYTAC_MDBT42Q-512KV2, F.Cu at (165.1, 99.1)
- moved C1 23.6 mm to (152.4, 88.9), turned to 0 degrees
- moved X1 21.0 mm to (152.4, 91.4), turned to 0 degrees
- moved C2 18.6 mm to (152.4, 94.0), turned to 180 degrees
- moved R1 2.66 mm to (123.7, 103.7)
- moved C11 2.66 mm to (123.7, 108.1)
- moved C15 2.66 mm to (133.9, 106.8)
- moved MAG1 2.66 mm to (128.8, 106.2)
- moved R2 2.66 mm to (126.9, 101.7)
- moved C10 2.14 mm to (157.5, 91.4), turned to 90 degrees
Connections:
- C10 pad 1: /DEC4 -> +3V3
- CVIN1 pad 1: +6V -> unconnected-(CVIN1-Pad1)
- CVOUT1 pad 1: +3V3 -> unconnected-(CVOUT1-Pad1)
- MAG1 pad 12: (no net) -> unconnected-(MAG1-Pad12)
- MAG1 pad 14: (no net) -> unconnected-(MAG1-Pad14)
- MAG1 pad 15: (no net) -> unconnected-(MAG1-Pad15)
- MAG1 pad 3: (no net) -> unconnected-(MAG1-Pad3)
- MAG1 pad 4: Net-(MAG1-Pad4) -> unconnected-(MAG1-Pad4)
- MAG1 pad 5: Net-(MAG1-Pad5) -> unconnected-(MAG1-Pad5)
- MAG1 pad 6: Net-(MAG1-Pad12) -> unconnected-(MAG1-Pad6)
- MAG1 pad 7: (no net) -> unconnected-(MAG1-Pad7)
- MAG1 pad 8: (no net) -> unconnected-(MAG1-Pad8)
- SD_SLOT1 pad 1: Net-(SD_SLOT1-Pad1) -> unconnected-(SD_SLOT1-Pad1)
- SD_SLOT1 pad 10: Net-(SD_SLOT1-Pad10) -> unconnected-(SD_SLOT1-Pad10)
- SD_SLOT1 pad 8: Net-(SD_SLOT1-Pad8) -> unconnected-(SD_SLOT1-Pad8)
- SD_SLOT1 pad 9: Net-(SD_SLOT1-Pad9) -> unconnected-(SD_SLOT1-Pad9)
- U_HB1 pad 1: Net-(U_HB1-Pad1) -> unconnected-(U_HB1-Pad1)
- U_HB1 pad 10: Net-(U_HB1-Pad10) -> unconnected-(U_HB1-Pad10)
- U_HB1 pad 14: Net-(U_HB1-Pad14) -> unconnected-(U_HB1-Pad14)
- U_HB1 pad 5: Net-(U_HB1-Pad5) -> unconnected-(U_HB1-Pad5)
Routing:
- net +3V3: track 93.2 -> 59.4 mm, vias 9 -> 6
- net /SCL: track 41.8 -> 13.8 mm
- net /MSCL: track 43.1 -> 19.4 mm, vias 1 -> 0
- net /INB: track 63.3 -> 41.7 mm
- net /DEC4: track 13.6 -> 0.00 mm
- net /XC1: track 13.3 -> 2.09 mm
- net Net-(MCU1-Pad4): track 10.6 -> 0.00 mm
- net /INA: track 63.9 -> 53.6 mm
- net Net-(MCU1-Pad3): track 10.2 -> 0.00 mm
- net /IND: track 61.9 -> 53.4 mm
- net /INC: track 61.9 -> 53.6 mm
- net /XC2: track 10.2 -> 2.09 mm
- net Net-(MCU1-Pad9): track 7.02 -> 0.00 mm
- net /WSS2: track 42.4 -> 35.4 mm
- net /SDA: track 32.8 -> 26.2 mm
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- removed copper zone on F.Cu, net /RF
- removed copper zone on F.Cu, net GND
Other:
- net class Default removed
- board text added: "ECE 477 Team 16"
