File: RepeatRoverV2.0/_autosave-RepeatRover.sch (KiCad schematic (older format))
At the start: 8 parts

Commit message: new mcu footgprint
Parts:
- removed h-bridge: YX-1818BM, symbol Interface_Expansion:PCA9516
- added C10, C_RST1: 1uF, Capacitor_SMD:C_0805_2012Metric_Pad1.18x1.45mm_HandSolder, symbol Device:C
- added C12, C16: 100uF, Capacitor_SMD:C_0805_2012Metric_Pad1.18x1.45mm_HandSolder, symbol Device:C
- added C13, C14: .1uF, Capacitor_SMD:C_0805_2012Metric_Pad1.18x1.45mm_HandSolder, symbol Device:C
- added C3: 0.8pF, Capacitor_SMD:C_0805_2012Metric_Pad1.18x1.45mm_HandSolder, symbol Device:C
- added C4, C5, C8: 100nF, Capacitor_SMD:C_0805_2012Metric_Pad1.18x1.45mm_HandSolder, symbol Device:C
- added C7: 100pF, Capacitor_SMD:C_0805_2012Metric_Pad1.18x1.45mm_HandSolder, symbol Device:C
- added C9: 4.7uF, Capacitor_SMD:C_0805_2012Metric_Pad1.18x1.45mm_HandSolder, symbol Device:C
- added CVIN1, CVOUT1: 10uF, Capacitor_SMD:CP_Elec_5x5.7, symbol Device:C_Polarized
- added H1, H2, H3, H4: MountingHole, MountingHole:MountingHole_3.2mm_M3, symbol Mechanical:MountingHole
- added J1, J2: Conn_01x02_Male, symbol Connector:Conn_01x02_Male
- added J1_1, J2_1: Conn_01x02_Female, Connector_PinSocket_2.54mm:PinSocket_1x02_P2.54mm_Vertical, symbol Connector:Conn_01x02_Female
- added J3, J4: Conn_01x03_Male, symbol Connector:Conn_01x03_Male
- added J3_1, J4_1: Conn_01x03_Female, Connector_PinSocket_2.54mm:PinSocket_1x03_P2.54mm_Vertical, symbol Connector:Conn_01x03_Female
- added J5: Barrel_Jack, Connector_BarrelJack:BarrelJack_CUI_PJ-102AH_Horizontal, symbol Connector:Barrel_Jack
- added L1: 3.9nH, Inductor_SMD:L_0402_1005Metric_Pad0.77x0.64mm_HandSolder, symbol Device:L
- added L2: 10uH, Inductor_SMD:L_0201_0603Metric_Pad0.64x0.40mm_HandSolder, symbol Device:L
- added L3: 15nH, Inductor_SMD:L_0402_1005Metric_Pad0.77x0.64mm_HandSolder, symbol Device:L
- added LDO1: NCP1117-3.3_SOT223, Package_TO_SOT_SMD:SOT-223-3_TabPin2, symbol Regulator_Linear:NCP1117-3.3_SOT223
- added M1, M2: Motor_DC, symbol Motor:Motor_DC
- added R1, R2: 2.7k, Resistor_SMD:R_0805_2012Metric_Pad1.20x1.40mm_HandSolder, symbol Device:R_US
- added R_RST1: 10k, Resistor_SMD:R_0805_2012Metric_Pad1.20x1.40mm_HandSolder, symbol Device:R_US
- added SW_RST1: _, Button_Switch_THT:SW_PUSH_6mm, symbol Switch:SW_Push
- added U_HB1: YX1818BM, Package_SO:SOP-16_4.55x10.3mm_P1.27mm, symbol HallEffect:YX1818BM
- added WSS1, WSS2: DRV5057, symbol HallEffect:DRV5057
- added X1: 32MHz, Hall Effect Footprint:OSC_XRCGB32M000FXH2CR0, symbol Device:Crystal
- C1, C2: value .1uF -> 12pF; footprint Capacitor_SMD:C_0805_2012Metric -> Capacitor_SMD:C_0805_2012Metric_Pad1.18x1.45mm_HandSolder
- C11: renamed from C1; footprint Capacitor_SMD:C_0805_2012Metric -> Capacitor_SMD:C_0805_2012Metric_Pad1.18x1.45mm_HandSolder
- C15: renamed from C2; footprint Capacitor_SMD:C_0805_2012Metric -> Capacitor_SMD:C_0805_2012Metric_Pad1.18x1.45mm_HandSolder
- renumbered MAG to MAG1, MCU to MCU1, SD_SLOT to SD_SLOT1
Connections:
- net labels added: +6V, ANT, DCC, DEC1, DEC2, DEC3, DEC4, EXP, INA, INB, INC, IND, MSCL, RF, SDCLK, SWDIO, VDD1, VDD2, VDD3, VSS1, VSS2, WSS1, WSS2, XC1, XC2, nRESET
- net labels removed: +3V0
- wire segments 43 -> 183
- no-connect marks 6 -> 4
Other:
- moved on the sheet: C11, C15, MAG1, SD_SLOT1
