File: RepeatRoverV2.0/MMCBreakOut/MMCBreakOut.kicad_pcb (KiCad board)
At the start: 2 copper layers, 31.8 x 11.4 mm, 7 parts, among them J1 _, J2 _

Commit message: new mcu footgprint
Parts:
- moved C2 11.8 mm to (106.7, 62.0)
Routing:
- net GND: track 20.6 -> 29.8 mm
- net +3V3: track 73.1 -> 76.8 mm
Other:
- net class Default removed
